Commit message: combined with rirolab complex_action_client, BT, and WM

File: art_med_robots_description/urdf/pioneer-lx-jaco2.urdf.xacro (robot description, xacro)
@@ -82,4 +82,5 @@
     </visual>
 -->
+<!--
     <collision name="r_wheel_collision">
       <geometry name="r_wheel_collision_geom">
@@ -88,4 +89,5 @@
       <origin rpy="1.570796 0 0" />
     </collision>
+-->
   </link>
   <!-- left wheel -->
@@ -106,4 +108,5 @@
     </visual>
    -->
+<!--
     <collision name="l_wheel_collision">
       <geometry name="l_wheel_collision_geom">
@@ -112,4 +115,5 @@
       <origin rpy="1.570796 0 0" />
     </collision>
+-->
   </link>
   <!-- wheel joints. only used in gazebo, real robot velocity is controlled as a unit, not individual wheel motion. -->
@@ -161,5 +165,4 @@
 		  <mesh filename="package://amr_robots_description/meshes/pioneer-lx/pioneer-lx-plinth.stl" scale="0.001 0.001 0.001" />
         <!-- box size="0.18 0.2476 0.99" / -->
-        <origin xyz="-0.02 0 0.867" />
       </geometry>
     </collision>
@@ -195,3 +198,15 @@
   <xacro:j2n6s300  base_parent="left_arm_mount" prefix="left" />
   <xacro:j2n6s300  base_parent="right_arm_mount" prefix="right" />
+  <!-- PTU
+    The flir_ptu_description package is either from system packages in
+    /opt/ros/... or from source repository
+    https://github.com/ros-drivers/flir_ptu
+  -->
+  <xacro:include filename="$(find art_med_robots_description)/urdf/d46.urdf.xacro" />
+  <ptu_d46 name="ptu" />
+  <joint name="ptu_base_mount" type="fixed">
+    <parent link="plinth" />
+    <child link="ptu_base_link" />
+    <origin xyz="0.152 0.03 0.91" />
+  </joint>
 </robot>
